File: NailPrinter_PCB/NailPrinter_PCB.kicad_sch (KiCad schematic)
At the start: 0 parts

Commit message: Beginning PCB Design and ReadMe
Other:
- added sheet Smart_Carriage (Smart_Carriage.kicad_sch)
- added sheet Stationary_Mainboard (Stationary_Mainboard.kicad_sch)
Changed lines of the file:
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@@
 	(generator_version "10.0")
 	(paper "A4")
+	(sheet
+		(at 62.23 102.87)
+		(size 92.71 38.1)
+		(exclude_from_sim no)
+		(in_bom yes)
+		(on_board yes)
+		(dnp no)
+		(fields_autoplaced yes)
+		(stroke
+			(width 0.1524)
+			(type solid)
+		)
+		(fill
+			(color 0 0 0 0)
+		)
+		(property "Sheetname" "Smart_Carriage"
+			(at 62.23 102.1584 0)
+			(show_name no)
+			(do_not_autoplace no)
+			(effects
+				(font
+					(size 1.27 1.27)
+				)
+				(justify left bottom)
+			)
+		)
+		(property "Sheetfile" "Smart_Carriage.kicad_sch"
+			(at 62.23 141.5546 0)
+			(show_name no)
+			(do_not_autoplace no)
+			(effects
+				(font
+					(size 1.27 1.27)
+				)
+				(justify left top)
+			)
+		)
+		(instances
+			(project "NailPrinter_PCB"
+				(path "/876b3e30-d187-46f3-87a9-b93d7260baa1"
+					(page "3")
+				)
+			)
+		)
+	)
+	(sheet
+		(at 52.07 30.48)
+		(size 105.41 48.26)
+		(exclude_from_sim no)
+		(in_bom yes)
+		(on_board yes)
+		(dnp no)
+		(fields_autoplaced yes)
+		(stroke
+			(width 0.1524)
+			(type solid)
+		)
+		(fill
+			(color 0 0 0 0)
+		)
+		(property "Sheetname" "Stationary_Mainboard"
+			(at 52.07 29.7684 0)
+			(show_name no)
+			(do_not_autoplace no)
+			(effects
+				(font
+					(size 1.27 1.27)
+				)
+				(justify left bottom)
+			)
+		)
+		(property "Sheetfile" "Stationary_Mainboard.kicad_sch"
+			(at 52.07 79.3246 0)
+			(show_name no)
+			(do_not_autoplace no)
+			(effects
+				(font
+					(size 1.27 1.27)
+				)
+				(justify left top)
+			)
+		)
+		(instances
+			(project "NailPrinter_PCB"
+				(path "/876b3e30-d187-46f3-87a9-b93d7260baa1"
+					(page "2")
+				)
+			)
+		)
+	)
 	(sheet_instances
 		(path "/"
