File: NailPrinter_PCB/Smart_Carriage.kicad_sch (KiCad schematic)
At the start: 0 parts

Commit message: mostly schematic and pcb design
Parts:
- added C3, C4, C7, C8: 10n, Capacitor_SMD:C_0805_2012Metric, symbol Device:C
- added C5, C6: 100n, Capacitor_SMD:C_0805_2012Metric, symbol Device:C
- added C9: 100m, symbol Device:C
- added J10: Conn_01x24, Connector_IDC:IDC-Header_2x12_P2.54mm_Vertical, symbol Connector_Generic:Conn_01x24
- added Q1, Q2: AO3401, Package_TO_SOT_SMD:SOT-23, symbol AO3401:AO3401
- added R1, R5: 10k, Resistor_SMD:R_0805_2012Metric, symbol Device:R
- added R2, R3, R6, R7: 1k, Resistor_SMD:R_0805_2012Metric, symbol Device:R
- added R4, R8: 2.7, Resistor_SMD:R_0805_2012Metric, symbol Device:R
- added U2, U5: AO3400, Package_TO_SOT_SMD:SOT-23, symbol AO3400:AO3400
- added U3, U4: CD4504BM, Package_SO:SOIC-16_3.9x9.9mm_P1.27mm, symbol CD4504BM:CD4504BM
Connections:
- new net: C3.2, Q1.1, R3.2
- new net: Q1.3, R2.1, R3.1, R4.2
- new net: C7.1, R6.2, U5.3
- new net: C7.2, Q2.1, R7.2
- new net: Q2.3, R6.1, R7.1, R8.2
- new net: C3.1, R2.2, U2.3
- new net +16V: C9.1, J10.1 (Pin_1), J10.2 (Pin_2), J10.3 (Pin_3), R4.1, R8.1
- new net +3.3V: C5.1, J10.19 (Pin_19), U3.1 (VCC), U4.1 (VCC)
- new net +9V: C6.2, J10.8 (Pin_8), U3.16 (VDD), U4.16 (VDD)
- new net CLK_3V: J10.10 (Pin_10), U3.7 (CIN)
- new net CLK_9V: U3.6 (COUT)
- new net D1_3V: J10.12 (Pin_12), U3.11 (EIN)
- new net D1_9V: U3.12 (EOUT)
- new net D2_3V: J10.13 (Pin_13), U3.5 (BIN)
- new net D2_9V: U3.4 (BOUT)
- new net D3_3V: J10.14 (Pin_14), U3.9 (DIN)
- new net D3_9V: U3.10 (DOUT)
- new net D4_3V: J10.20 (Pin_20), U3.14 (FIN)
- new net D4_9V: U3.15 (FOUT)
- new net D5_3V: J10.21 (Pin_21), U4.3 (AIN)
- new net D5_9V: U4.2 (AOUT)
- new net D6_3V: J10.22 (Pin_22), U4.5 (BIN)
- new net D6_9V: U4.4 (BOUT)
- new net D7_3V: J10.23 (Pin_23), U4.7 (CIN)
- new net D7_9V: U4.6 (COUT)
- new net D8_3V: J10.24 (Pin_24), U4.9 (DIN)
- new net D8_9V: U4.10 (DOUT)
- new net ENC_A: J10.16 (Pin_16)
- new net ENC_B: J10.17 (Pin_17)
- new net GND: C4.1, C5.2, C6.1, C8.1, C9.2, J10.11 (Pin_11), J10.15 (Pin_15), J10.18 (Pin_18), J10.4 (Pin_4), J10.7 (Pin_7), R1.2, R5.2, U2.2, U3.13 (SELECT), U3.8 (VSS), U4.11 (EIN), U4.13 (SELECT), U4.14 (FIN), U4.8 (VSS), U5.2
- new net PWRA_IN: J10.6 (Pin_6), R1.1, U2.1
- new net PWRA_OUT: C4.2, Q1.2
- new net PWRB_IN: J10.5 (Pin_5), R5.1, U5.1
- new net PWRB_OUT: C8.2, Q2.2
- new net SYNC_3V: J10.9 (Pin_9), U3.3 (AIN)
- new net SYNC_9V: U3.2 (AOUT)
- no-connect marks 0 -> 2
