File: NailPrinter_PCB/NailPrinter_PCB.kicad_pcb (KiCad board)
At the start: 2 copper layers, 233.5 x 103 mm, 37 parts, among them J1 Barrel_Jack, J10 Conn_01x24, J2 Conn_01x03, J3 Conn_01x04, J4 Conn_01x04, J5 Conn_01x04, J6 Conn_01x04, J7 Conn_01x03, J8 Conn_01x04, J9 Conn_01x24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

Commit message: Preliminary traces, probably needs a lot more tweaking
Parts:
- removed J7: Conn_01x03, Connector_JST:JST_XH_B3B-XH-A_1x03_P2.50mm_Vertical
- moved U1 15.7 mm to (44.8, 69.0)
- moved C2 5.70 mm to (68.5, 127.5), turned to 90 degrees
- moved C1 2.69 mm to (76.5, 127.0), turned to 90 degrees
- moved U_TMC_Y1 0.75 mm to (40.7, 113.1)
Routing:
- net +3.3V: track 0.00 -> 173.2 mm
- net +16V: track 0.00 -> 156.5 mm
- net +5V: track 0.00 -> 108.4 mm
- net +9V: track 0.00 -> 96.1 mm
- net CLK_3V: track 0.00 -> 92.5 mm
- net D1_3V: track 0.00 -> 84.3 mm
- net D2_3V: track 0.00 -> 79.0 mm
- net +24V: track 0.00 -> 78.2 mm
- net D3_3V: track 0.00 -> 76.5 mm
- net D4_3V: track 0.00 -> 65.3 mm
- net D5_3V: track 0.00 -> 64.5 mm
- net PWRA_IN: track 0.00 -> 58.9 mm
- net D6_3V: track 0.00 -> 58.6 mm
- net ENC_A: track 0.00 -> 52.5 mm
- net ENC_B: track 0.00 -> 52.4 mm
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